File: PCB/RobotHand.kicad_pcb (KiCad board)
At the start: 2 copper layers, 121.9 x 124.7 mm, 29 parts, among them J1 Screw_Terminal_01x02, U1 ADS7830, U3 DRV8835DSSR, U5 DRV8835DSSR, U6 DRV8835DSSR

Commit message: Version 2 of PCB
Parts:
- removed EXT_ADC_CH1: Conn_01x08_Pin, Connector_PinHeader_2.54mm:PinHeader_1x08_P2.54mm_Vertical
- added C10: 0.1uF, Capacitor_SMD:C_0805_2012Metric_Pad1.18x1.45mm_HandSolder, F.Cu at (112.5, 137.9)
- added C11: 0.1uF, Capacitor_SMD:C_0805_2012Metric_Pad1.18x1.45mm_HandSolder, F.Cu at (108.0, 141.0)
- added C4: 0.1uF, Capacitor_SMD:C_0805_2012Metric_Pad1.18x1.45mm_HandSolder, F.Cu at (112.0, 76.5)
- added C6: 0.1uF, Capacitor_SMD:C_0805_2012Metric_Pad1.18x1.45mm_HandSolder, F.Cu at (78.0, 92.2)
- added C7: 0.1uF, Capacitor_SMD:C_0805_2012Metric_Pad1.18x1.45mm_HandSolder, F.Cu at (108.0, 136.4)
- added C8: 0.1uF, Capacitor_SMD:C_0805_2012Metric_Pad1.18x1.45mm_HandSolder, F.Cu at (115.8, 72.9)
- added C9: 0.1uF, Capacitor_SMD:C_0805_2012Metric_Pad1.18x1.45mm_HandSolder, F.Cu at (80.0, 87.6)
- added D1: D_Zener, Diode_SMD:D_SOD-123, F.Cu at (101.1, 145.3)
- added H1: MountingHole, MountingHole:MountingHole_6.4mm_M6, F.Cu at (52.1, 66.3)
- added H2: MountingHole, MountingHole:MountingHole_6.4mm_M6, F.Cu at (157.5, 47.2)
- added H3: MountingHole, MountingHole:MountingHole_6.4mm_M6, F.Cu at (86.9, 152.7)
- added J2: Conn_01x07_Pin, Connector_PinSocket_2.54mm:PinSocket_1x07_P2.54mm_Vertical, F.Cu at (149.9, 78.7)
- added Q1: PMOS, Package_TO_SOT_SMD:SOT-23-3, F.Cu at (108.1, 146.8)
- added R1: 100k, Resistor_SMD:R_0805_2012Metric, F.Cu at (113.8, 146.8)
- C1, C2, C3: footprint Capacitor_SMD:C_0805_2012Metric -> Capacitor_SMD:C_0805_2012Metric_Pad1.18x1.45mm_HandSolder
- C5: value 0.1uF -> 100uF; footprint Capacitor_SMD:C_0805_2012Metric -> Capacitor_SMD:C_0805_2012Metric_Pad1.18x1.45mm_HandSolder
- R2, R3: value 10k -> 4.7k
- moved C2 23.4 mm to (123.7, 77.0)
- moved U1 22.5 mm to (131.2, 81.3)
- moved C5 19.5 mm to (102.1, 139.4), turned to 0 degrees
- moved J1 10.2 mm to (109.2, 154.7)
- moved U3 8.68 mm to (73.2, 86.6), turned to -90 degrees
- moved C1 8.57 mm to (109.0, 116.1), turned to 35 degrees
- moved R2 7.94 mm to (92.7, 111.0), turned to -50 degrees
- moved R3 7.58 mm to (96.5, 108.2), turned to -50 degrees
- moved U2 6.45 mm to (92.0, 119.3), turned to 125 degrees
- moved C3 5.91 mm to (104.1, 115.6), turned to -145 degrees
- moved ThumbConnector1 2.79 mm to (138.3, 121.9), turned to -25 degrees
- moved PalmPot1 2.34 mm to (140.9, 103.6)
- moved Middle_01 1.69 mm to (93.2, 65.0)
- moved Ring_01 1.61 mm to (62.5, 58.9)
- moved U6 1.50 mm to (109.2, 72.5)
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Connections:
- C5 pad 1: GND -> Net-(D1-A)
- C5 pad 2: V_BATT -> GND
- IndexPot1 pad 2: ADC_CH0 -> ADC_CH1
- J1 pad 1: V_BATT -> Net-(J1-Pin_1)
- MiddlePot1 pad 2: ADC_CH1 -> ADC_CH4
- PalmPot1 pad 2: ADC_CH5 -> ADC_CH2
- RingPot1 pad 2: ADC_CH2 -> ADC_CH5
- ThumbConnector1 pad 2: ADC_CH4 -> ADC_CH0
- U1 pad 7: Net-(EXT_ADC_CH1-Pin_7) -> GND
- U1 pad 8: Net-(EXT_ADC_CH1-Pin_8) -> GND
- U2 pad 10: unconnected-(U2-IO2-Pad10) -> Thumb_EN
- U2 pad 21: Middle_EN -> Index_PH
- U2 pad 22: Middle_PH -> Index_EN
- U2 pad 23: Index_EN -> Middle_PH
- U2 pad 24: Index_PH -> Middle_EN
- U2 pad 3: Palm_PH -> Ring_EN
- U2 pad 32: Ring_PH -> unconnected-(U2-IO15-Pad32)
- U2 pad 33: Ring_EN -> unconnected-(U2-In35-Pad33)
- U2 pad 4: Palm_EN -> Ring_PH
- U2 pad 5: Thumb_PH -> Palm_PH
- U2 pad 6: Thumb_EN -> unconnected-(U2-IO9^{SPIF}-Pad6)
- U2 pad 8: unconnected-(U2-IO13-Pad8) -> Palm_EN
- U2 pad 9: unconnected-(U2-IO5-Pad9) -> Thumb_PH
- U3 pad 1: V_BATT -> Net-(U3-VM)
- U3 pad 12: VDD -> Net-(U3-VCC)
- U5 pad 1: V_BATT -> Net-(U5-VM)
- U5 pad 12: VDD -> Net-(U5-VCC)
- U6 pad 1: V_BATT -> Net-(U6-VM)
- U6 pad 12: VDD -> Net-(U6-VCC)
Routing:
- net ADC_CH5: track 44.2 -> 90.2 mm
- net Index_PH: track 58.4 -> 29.5 mm
- net ADC_CH4: track 68.3 -> 41.5 mm, vias 2 -> 0
- net ADC_CH3: track 69.5 -> 96.0 mm, vias 4 -> 6
- net ADC_CH0: track 39.2 -> 64.8 mm, vias 2 -> 4
- net Pinkie_EN: track 51.1 -> 26.2 mm
- net Index_EN: track 55.8 -> 31.6 mm
- net GND: track 30.5 -> 54.3 mm, vias 4 -> 6
- net Pinkie_PH: track 47.6 -> 27.1 mm
- net Middle_PH: track 54.2 -> 33.8 mm
- net Net-(EXT_ADC_CH1-Pin_8): track 19.9 -> 0.00 mm
- net Net-(EXT_ADC_CH1-Pin_7): track 18.5 -> 0.00 mm
- net Middle_EN: track 52.6 -> 35.9 mm
- net Net-(Pinkie_02-Pin_1): track 47.9 -> 35.0 mm, vias 0 -> 2
- net VDD: track 300.1 -> 311.8 mm, vias 10 -> 12
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Other:
- outline, holes or cut-outs redrawn
- board text added: "+"
- board text added: "C"
- board text added: "For Instructional Use Only."
- board text added: "GND"
- board text added: "Index_01"
- board text added: "Index_02"
- board text added: "Middle_01"
- board text added: "Middle_02"
- board text added: "Palm_01"
- board text added: "Palm_02"
- board text added: "Pinkie_01"
- board text added: "Pinkie_02"
- board text added: "Ring_01"
- board text added: "Ring_02"
- board text added: "SOLIDWORKS Educational Product."
- board text added: "VDD ADC GND 01 02"
