File: PCB/RobotHand.kicad_sch (KiCad schematic)
At the start: 30 parts, among them J1 Screw_Terminal_01x02, U1 ADS7830, U3 DRV8835DSSR, U4 ESP32-WROOM-32D, U5 DRV8835DSSR, U6 DRV8835DSSR

Commit message: Added footprints to first PCB version
Parts:
- C1, C2, C3, C4, C5: footprint (none) -> Capacitor_SMD:C_0805_2012Metric
- EXT_ADC_CH: footprint (none) -> Connector_PinHeader_2.54mm:PinHeader_1x08_P2.54mm_Vertical
- Index_01, Index_02, Middle_01, Middle_02, Palm_01, Palm_02, Pinkie_01, Pinkie_02, Ring_01, Ring_02, Thumb_01, Thumb_02: footprint (none) -> Connector_PinHeader_2.54mm:PinHeader_1x01_P2.54mm_Vertical
- J1: footprint (none) -> TerminalBlock:TerminalBlock_Xinya_XY308-2.54-2P_1x02_P2.54mm_Horizontal
- R1, R2, R3: footprint (none) -> Resistor_SMD:R_0805_2012Metric
- RotaryPot1, RotaryPot2, RotaryPot3: footprint (none) -> Connector_PinHeader_2.54mm:PinHeader_1x03_P2.54mm_Vertical
Changed lines of the file:
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@@
 			)
 		)
-		(property "Footprint" ""
+		(property "Footprint" "Connector_PinHeader_2.54mm:PinHeader_1x01_P2.54mm_Vertical"
 			(at 251.46 96.52 0)
 			(effects
@@
 			)
 		)
-		(property "Footprint" ""
+		(property "Footprint" "Connector_PinHeader_2.54mm:PinHeader_1x01_P2.54mm_Vertical"
 			(at 251.46 35.56 0)
 			(effects
@@
 			)
 		)
-		(property "Footprint" ""
+		(property "Footprint" "Connector_PinHeader_2.54mm:PinHeader_1x01_P2.54mm_Vertical"
 			(at 252.73 137.16 0)
 			(effects
@@
 			)
 		)
-		(property "Footprint" ""
+		(property "Footprint" "Connector_PinHeader_2.54mm:PinHeader_1x01_P2.54mm_Vertical"
 			(at 251.46 43.18 0)
 			(effects
@@
 			)
 		)
-		(property "Footprint" ""
+		(property "Footprint" "Resistor_SMD:R_0805_2012Metric"
 			(at 42.418 147.32 90)
 			(effects
@@
 			)
 		)
-		(property "Footprint" ""
+		(property "Footprint" "Resistor_SMD:R_0805_2012Metric"
 			(at 24.892 147.32 90)
 			(effects
@@
 			)
 		)
-		(property "Footprint" ""
+		(property "Footprint" "Connector_PinHeader_2.54mm:PinHeader_1x01_P2.54mm_Vertical"
 			(at 251.46 86.36 0)
 			(effects
@@
 			)
 		)
-		(property "Footprint" ""
+		(property "Footprint" "Connector_PinHeader_2.54mm:PinHeader_1x03_P2.54mm_Vertical"
 			(at 140.97 81.28 0)
 			(effects
@@
 			)
 		)
-		(property "Footprint" ""
+		(property "Footprint" "Connector_PinHeader_2.54mm:PinHeader_1x01_P2.54mm_Vertical"
 			(at 252.73 147.32 0)
 			(effects
@@
 			)
 		)
-		(property "Footprint" ""
+		(property "Footprint" "Connector_PinHeader_2.54mm:PinHeader_1x01_P2.54mm_Vertical"
 			(at 251.46 93.98 0)
 			(effects
@@
 			)
 		)
-		(property "Footprint" ""
+		(property "Footprint" "Connector_PinHeader_2.54mm:PinHeader_1x08_P2.54mm_Vertical"
 			(at 22.86 80.01 0)
 			(effects
@@
 			)
 		)
-		(property "Footprint" ""
+		(property "Footprint" "Capacitor_SMD:C_0805_2012Metric"
 			(at 88.9 33.3248 0)
 			(effects
@@
 			)
 		)
-		(property "Footprint" ""
+		(property "Footprint" "TerminalBlock:TerminalBlock_Xinya_XY308-2.54-2P_1x02_P2.54mm_Horizontal"
 			(at 140.97 134.62 0)
 			(effects
@@
 			)
 		)
-		(property "Footprint" ""
+		(property "Footprint" "Connector_PinHeader_2.54mm:PinHeader_1x01_P2.54mm_Vertical"
 			(at 252.73 139.7 0)
 			(effects
@@
 			)
 		)
-		(property "Footprint" ""
+		(property "Footprint" "Connector_PinHeader_2.54mm:PinHeader_1x03_P2.54mm_Vertical"
 			(at 140.97 91.44 0)
 			(effects
@@
 			)
 		)
-		(property "Footprint" ""
+		(property "Footprint" "Resistor_SMD:R_0805_2012Metric"
 			(at 31.75 24.638 90)
 			(effects
@@
 			)
 		)
-		(property "Footprint" ""
+		(property "Footprint" "Connector_PinHeader_2.54mm:PinHeader_1x01_P2.54mm_Vertical"
 			(at 251.46 40.64 0)
 			(effects
@@
 			)
 		)
-		(property "Footprint" ""
+		(property "Footprint" "Connector_PinHeader_2.54mm:PinHeader_1x03_P2.54mm_Vertical"
 			(at 140.97 101.6 0)
 			(effects
@@
 			)
 		)
-		(property "Footprint" ""
+		(property "Footprint" "Connector_PinHeader_2.54mm:PinHeader_1x01_P2.54mm_Vertical"
 			(at 251.46 88.9 0)
 			(effects
@@
 			)
 		)
-		(property "Footprint" ""
+		(property "Footprint" "Capacitor_SMD:C_0805_2012Metric"
 			(at 103.8352 67.31 0)
 			(effects
@@
 			)
 		)
-		(property "Footprint" ""
+		(property "Footprint" "Connector_PinHeader_2.54mm:PinHeader_1x01_P2.54mm_Vertical"
 			(at 252.73 144.78 0)
 			(effects
@@
 			)
 		)
-		(property "Footprint" ""
+		(property "Footprint" "Connector_PinHeader_2.54mm:PinHeader_1x01_P2.54mm_Vertical"
 			(at 251.46 33.02 0)
 			(effects
@@
 			)
 		)
-		(property "Footprint" ""
+		(property "Footprint" "Capacitor_SMD:C_0805_2012Metric"
 			(at 53.0352 34.29 0)
 			(effects
@@
 			)
 		)
-		(property "Footprint" ""
+		(property "Footprint" "Capacitor_SMD:C_0805_2012Metric"
 			(at 119.6848 137.16 0)
 			(effects
@@
 			)
 		)
-		(property "Footprint" ""
+		(property "Footprint" "Capacitor_SMD:C_0805_2012Metric"
 			(at 40.3352 34.29 0)
 			(effects

Commit message: First revision of pcb design
Parts:
- removed C4: 10uF, Capacitor_SMD:C_0805_2012Metric, symbol Device:C
- removed R1: 5, Resistor_SMD:R_0805_2012Metric, symbol Device:R
- removed Thumb_01, Thumb_02: Conn_01x01, Connector_PinHeader_2.54mm:PinHeader_1x01_P2.54mm_Vertical, symbol Connector_Generic:Conn_01x01
- removed U4: ESP32-WROOM-32D, RF_Module:ESP32-WROOM-32D, symbol RF_Module:ESP32-WROOM-32D
- added PalmPot1, PinkiePot1: Conn_01x03, Connector_PinHeader_2.54mm:PinHeader_1x03_P2.54mm_Vertical, symbol Connector_Generic:Conn_01x03
- added ThumbConnector1: Conn_01x05, Connector_PinHeader_2.54mm:PinHeader_1x05_P2.54mm_Vertical, symbol Connector_Generic:Conn_01x05
- added U2: ~, ME507F24:FireBeetle-ESP32, symbol ME507F24:FireBeetle-ESP32
- U3, U5, U6: footprint DRV8835DSSR:SON50P300X200X80-13N -> Package_SON:WSON-12-1EP_3x2mm_P0.5mm_EP1x2.65
- renumbered EXT_ADC_CH to EXT_ADC_CH1, RotaryPot1 to IndexPot1, RotaryPot2 to MiddlePot1, RotaryPot3 to RingPot1
Connections:
- net GND: now also C1.1, PalmPot1.3 (Pin_3), PinkiePot1.3 (Pin_3), ThumbConnector1.3 (Pin_3), U2.15 (GND); no longer C1.2
- net Index_EN: now also U6.9 (AIN2/AENBL), U2.23 (MCLK/IO12); no longer U6.7 (BIN2/BENBL)
- net Index_PH: now also U6.10 (AIN1/APHASE), U2.24 (BCLK/IO14); no longer U6.8 (BIN1/BPHASE)
- net Middle_EN: now also U6.7 (BIN2/BENBL), U2.21 (DI/IO16); no longer U3.7 (BIN2/BENBL)
- net Middle_PH: now also U6.8 (BIN1/BPHASE), U2.22 (DO/IO4); no longer U3.8 (BIN1/BPHASE)
- net Palm_EN: now also U2.4 (IO26)
- net Palm_PH: now also U2.3 (IO25)
- net Pinkie_EN: now also U3.9 (AIN2/AENBL), U2.28 (MOSI/IO23); no longer U5.7 (BIN2/BENBL)
- net Pinkie_PH: now also U3.10 (AIN1/APHASE), U2.27 (MISO/IO19); no longer U5.8 (BIN1/BPHASE)
- net Ring_EN: now also U3.7 (BIN2/BENBL), U2.33 (In35); no longer U3.9 (AIN2/AENBL)
- net Ring_PH: now also U3.8 (BIN1/BPHASE), U2.32 (IO15); no longer U3.10 (AIN1/APHASE)
- net SCK: now also R3.1, U2.25 (SCL/IO22); no longer R2.2
- net SDA: now also R2.1, U2.26 (SDA/IO21); no longer R3.1
- net Thumb_EN: now also U5.7 (BIN2/BENBL), U2.6 (IO9^{SPIF}); no longer U6.9 (AIN2/AENBL)
- net Thumb_PH: now also U5.8 (BIN1/BPHASE), U2.5 (IO27); no longer U6.10 (AIN1/APHASE)
- net VDD: now also C1.2, C3.1, R2.2, PalmPot1.1 (Pin_1), PinkiePot1.1 (Pin_1), ThumbConnector1.1 (Pin_1), U2.17 (3V3); no longer C1.1, R2.1
- net at Middle_02.1 (Pin_1): now also U6.5 (BOUT2); no longer U3.5 (BOUT2)
- net at U6.3 (AOUT2): now also Index_02.1 (Pin_1)
- net at U6.2 (AOUT1): now also Index_01.1 (Pin_1)
- net at U6.4 (BOUT1): now also Middle_01.1 (Pin_1); no longer Index_01.1 (Pin_1)
- net at Ring_01.1 (Pin_1): now also U3.4 (BOUT1); no longer U3.2 (AOUT1)
- net at Pinkie_02.1 (Pin_1): now also U3.3 (AOUT2); no longer U5.5 (BOUT2)
- net at Pinkie_01.1 (Pin_1): now also U3.2 (AOUT1); no longer U5.4 (BOUT1)
- net ADC_CH3: now reaches EXT_ADC_CH1.4 (Pin_4), U1.4 (CH3)
- net ADC_CH3: now also PinkiePot1.2 (Pin_2)
- net ADC_CH4: now reaches EXT_ADC_CH1.5 (Pin_5), U1.5 (CH4)
- net ADC_CH4: now also ThumbConnector1.2 (Pin_2)
- net ADC_CH5: now reaches EXT_ADC_CH1.6 (Pin_6), U1.6 (CH5)
- net ADC_CH5: now also PalmPot1.2 (Pin_2)
- net at Ring_02.1 (Pin_1): now also U3.5 (BOUT2); no longer U3.3 (AOUT2)
- new net Thumb_01: ThumbConnector1.4 (Pin_4), U5.5 (BOUT2)
- new net Thumb_02: ThumbConnector1.5 (Pin_5), U5.4 (BOUT1)
Other:
- moved on the sheet: C1, C3, C5, IndexPot1, Index_01, Index_02, J1, MiddlePot1, Middle_01, Middle_02, Pinkie_01, Pinkie_02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

Commit message: Version 2 of PCB
Parts:
- removed EXT_ADC_CH1: Conn_01x08_Pin, Connector_PinHeader_2.54mm:PinHeader_1x08_P2.54mm_Vertical, symbol Connector:Conn_01x08_Pin
- added C10, C11, C4, C6, C7, C8, C9: 0.1uF, Capacitor_SMD:C_0805_2012Metric_Pad1.18x1.45mm_HandSolder, symbol Device:C
- added D1: D_Zener, Diode_SMD:D_SOD-123, symbol Device:D_Zener
- added H1, H2, H3: MountingHole, MountingHole:MountingHole_6.4mm_M6, symbol Mechanical:MountingHole
- added J2: Conn_01x07_Pin, Connector_PinSocket_2.54mm:PinSocket_1x07_P2.54mm_Vertical, symbol Connector:Conn_01x07_Pin
- added Q1: PMOS, Package_TO_SOT_SMD:SOT-23-3, symbol Simulation_SPICE:PMOS
- added R1: 100k, Resistor_SMD:R_0805_2012Metric, symbol Device:R
- C1, C2, C3: footprint Capacitor_SMD:C_0805_2012Metric -> Capacitor_SMD:C_0805_2012Metric_Pad1.18x1.45mm_HandSolder
- C5: value 0.1uF -> 100uF; footprint Capacitor_SMD:C_0805_2012Metric -> Capacitor_SMD:C_0805_2012Metric_Pad1.18x1.45mm_HandSolder
- R2, R3: value 10k -> 4.7k
Connections:
- net ADC_CH0: now also ThumbConnector1.2 (Pin_2), J2.1 (Pin_1); no longer IndexPot1.2 (Pin_2)
- net ADC_CH1: now also IndexPot1.2 (Pin_2), J2.2 (Pin_2); no longer MiddlePot1.2 (Pin_2)
- net ADC_CH2: now also PalmPot1.2 (Pin_2), J2.3 (Pin_3); no longer RingPot1.2 (Pin_2)
- net ADC_CH3: now also J2.4 (Pin_4)
- net ADC_CH4: now also MiddlePot1.2 (Pin_2), J2.5 (Pin_5); no longer ThumbConnector1.2 (Pin_2)
- net ADC_CH5: now also RingPot1.2 (Pin_2), J2.6 (Pin_6); no longer PalmPot1.2 (Pin_2)
- net GND: now also C5.2, U1.7 (CH6), U1.8 (CH7), C11.2, J2.7 (Pin_7), R1.2; no longer C5.1
- net Index_EN: now also U2.22 (DO/IO4); no longer U2.23 (MCLK/IO12)
- net Index_PH: now also U2.21 (DI/IO16); no longer U2.24 (BCLK/IO14)
- net Middle_EN: now also U2.24 (BCLK/IO14); no longer U2.21 (DI/IO16)
- net Middle_PH: now also U2.23 (MCLK/IO12); no longer U2.22 (DO/IO4)
- net Palm_EN: now also U2.8 (IO13); no longer U2.4 (IO26)
- net Palm_PH: now also U2.5 (IO27); no longer U2.3 (IO25)
- net Ring_EN: now also U2.3 (IO25); no longer U2.33 (In35)
- net Ring_PH: now also U2.4 (IO26); no longer U2.32 (IO15)
- net Thumb_EN: now also U2.10 (IO2); no longer U2.6 (IO9^{SPIF})
- net Thumb_PH: now also U2.9 (IO5); no longer U2.5 (IO27)
- net VDD: now also C4.2, C6.2, C7.2; no longer U3.12 (VCC), U5.12 (VCC), U6.12 (VCC)
- net V_BATT: now also C10.1, C11.1, C8.2, C9.2, D1.1 (K), Q1.3 (S); no longer C5.2, J1.1 (Pin_1), U3.1 (VM), U5.1 (VM), U6.1 (VM)
- new net: J1.1 (Pin_1), Q1.1 (D)
- new net: Q1.2 (G), R1.1
- new net: C8.1, U6.1 (VM)
- new net: C4.1, U6.12 (VCC)
- new net: C6.1, U3.12 (VCC)
- new net: C7.1, U5.12 (VCC)
- new net: C10.2, U5.1 (VM)
- new net: C5.1, D1.2 (A)
- new net: C9.1, U3.1 (VM)
Other:
- moved on the sheet: C1, C2, C3, C5, J1, U1
